File: Indication_ADUM.kicad_sch (KiCad schematic)
At the start: 25 parts

Commit message: Одна стойка
Connections:
- net FAULT renamed FAULT_1
- net READY_H renamed RDY_H1
- net READY_L renamed RDY_L1
- net ~{FAULT_H} renamed FLT_H1
- net ~{FAULT_L} renamed FLT_L1
