File: NTC_Handler.kicad_sch (KiCad schematic)
At the start: 0 parts

Commit message: Почти финальная версия
Parts:
- added U?: LM397, Package_TO_SOT_SMD:SOT-23-5, symbol Comparator:LM397
Changed lines of the file:
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@@
 (kicad_sch (version 20211123) (generator eeschema)
   (paper "A4")
+  (symbol (lib_id "Comparator:LM397") (at 149.098 96.139 0) (unit 1)
+    (in_bom yes) (on_board yes) (fields_autoplaced)
+    (property "Reference" "U?" (id 0) (at 158.75 91.44 0))
+    (property "Value" "LM397" (id 1) (at 158.75 93.98 0))
+    (property "Footprint" "Package_TO_SOT_SMD:SOT-23-5" (id 2) (at 150.368 111.379 0)
+      (effects (font (size 1.27 1.27)) hide)
+    )
+    (property "Datasheet" "http://www.ti.com/lit/ds/symlink/lm397.pdf" (id 3) (at 149.098 91.059 0)
+      (effects (font (size 1.27 1.27)) hide)
+    )
+    (pin "1")
+    (pin "2")
+    (pin "3")
+    (pin "4")
+    (pin "5")
+  )
 )
