File: Driver_SKiM459GD12E4 V2.kicad_sch (KiCad schematic)
At the start: 33 parts, among them J13 EL1, J14 GL1, J15 NTC1_A, J16 NTC1_B, J17 GH1, J18 OUT1, J19 CH1, J20 EL2, J21 GL2, J22 NTC2_A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

Commit message: Одна стойка
Other:
- added sheet Supply_Power (Supply_Power.kicad_sch)
Changed lines of the file:
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@@
+    )
+  )
+  (sheet (at 223.266 55.372) (size 28.194 22.352) (fields_autoplaced)
+    (stroke (width 0.1524) (type solid) (color 0 0 0 0))
+    (fill (color 0 0 0 0.0000))
+    (property "Sheet name" "Supply_Power" (id 0) (at 223.266 54.6604 0)
+      (effects (font (size 1.27 1.27)) (justify left bottom))
+    )
+    (property "Sheet file" "Supply_Power.kicad_sch" (id 1) (at 223.266 78.3086 0)
+      (effects (font (size 1.27 1.27)) (justify left top))
     )
   )
@@
     (path "/d88efb4f-8308-49e6-9154-1da2ad8b0e37" (page "3"))
     (path "/8479a9cb-eb9a-492e-bb8a-963500a48926" (page "4"))
+    (path "/f75c0da5-ea98-45b1-9a07-415549f295ff" (page "5"))
   )
   (symbol_instances
@@
       (reference "#PWR046") (unit 1) (value "+5VD") (footprint "")
     )
+    (path "/f75c0da5-ea98-45b1-9a07-415549f295ff/ff8f10f1-2154-46b8-8f4a-e12f7db0b0ce"
+      (reference "#PWR047") (unit 1) (value "+15V") (footprint "")
+    )
+    (path "/f75c0da5-ea98-45b1-9a07-415549f295ff/62cbe3ab-e755-4286-8185-c02c8630b294"
+      (reference "#PWR048") (unit 1) (value "GND3") (footprint "")
+    )
+    (path "/f75c0da5-ea98-45b1-9a07-415549f295ff/b67f28df-bd75-45f6-bcc6-898537ee41de"
+      (reference "#PWR049") (unit 1) (value "+15V") (footprint "")
+    )
+    (path "/f75c0da5-ea98-45b1-9a07-415549f295ff/caf8508d-8fdc-4a66-b72b-dad1f981b084"
+      (reference "#PWR050") (unit 1) (value "GND3") (footprint "")
+    )
     (path "/90ad37b3-1964-4d46-be98-f2e705808058/e4d1155b-8d60-47c7-aff5-45500bd95234"
       (reference "C1") (unit 1) (value "0.1u") (footprint "Capacitor_SMD:C_0805_2012Metric_Pad1.18x1.45mm_HandSolder")
@@
       (reference "C18") (unit 1) (value "56p") (footprint "Capacitor_SMD:C_0805_2012Metric_Pad1.18x1.45mm_HandSolder")
     )
+    (path "/f75c0da5-ea98-45b1-9a07-415549f295ff/70e996e7-ad33-48ea-add7-02444be2b34f"
+      (reference "C19") (unit 1) (value "10u") (footprint "Capacitor_SMD:C_1210_3225Metric_Pad1.33x2.70mm_HandSolder")
+    )
+    (path "/f75c0da5-ea98-45b1-9a07-415549f295ff/cc28e310-0e96-4de1-b7c9-1872ab94f355"
+      (reference "C20") (unit 1) (value "10u") (footprint "Capacitor_SMD:C_1210_3225Metric_Pad1.33x2.70mm_HandSolder")
+    )
+    (path "/90ad37b3-1964-4d46-be98-f2e705808058/8b6e897a-69ad-468a-b1a1-f26ad2399337"
+      (reference "C21") (unit 1) (value "1u") (footprint "Capacitor_SMD:C_0805_2012Metric_Pad1.18x1.45mm_HandSolder")
+    )
+    (path "/90ad37b3-1964-4d46-be98-f2e705808058/06df9233-8418-4488-837f-f27078d61b36"
+      (reference "C22") (unit 1) (value "1u") (footprint "Capacitor_SMD:C_0805_2012Metric_Pad1.18x1.45mm_HandSolder")
+    )
+    (path "/f75c0da5-ea98-45b1-9a07-415549f295ff/3874bad0-6962-418d-a123-c0dbddde79ee"
+      (reference "C23") (unit 1) (value "10u") (footprint "Capacitor_SMD:C_1210_3225Metric_Pad1.33x2.70mm_HandSolder")
+    )
+    (path "/f75c0da5-ea98-45b1-9a07-415549f295ff/33dbdc2c-9b2e-4936-ba2d-ff38d8b88e68"
+      (reference "C24") (unit 1) (value "10u") (footprint "Capacitor_SMD:C_1210_3225Metric_Pad1.33x2.70mm_HandSolder")
+    )
+    (path "/f75c0da5-ea98-45b1-9a07-415549f295ff/b24fbfce-8572-4f0d-ae84-b967e778238d"
+      (reference "C25") (unit 1) (value "10u") (footprint "Capacitor_SMD:C_1210_3225Metric_Pad1.33x2.70mm_HandSolder")
+    )
+    (path "/f75c0da5-ea98-45b1-9a07-415549f295ff/c834f2df-f5df-4e9c-9845-46586882a5d6"
+      (reference "C26") (unit 1) (value "10u") (footprint "Capacitor_SMD:C_1210_3225Metric_Pad1.33x2.70mm_HandSolder")
+    )
+    (path "/90ad37b3-1964-4d46-be98-f2e705808058/54c71382-e512-4277-9d3b-2fa3ffd2ad7a"
+      (reference "C27") (unit 1) (value "1u") (footprint "Capacitor_SMD:C_0805_2012Metric_Pad1.18x1.45mm_HandSolder")
+    )
+    (path "/90ad37b3-1964-4d46-be98-f2e705808058/fa1ece2f-9dc0-4fdc-af84-c71322678a04"
+      (reference "C28") (unit 1) (value "1u") (footprint "Capacitor_SMD:C_0805_2012Metric_Pad1.18x1.45mm_HandSolder")
+    )
     (path "/90ad37b3-1964-4d46-be98-f2e705808058/89aad84a-99b2-4cff-9a18-0bcef9ff760f"
       (reference "D1") (unit 1) (value "ADUM4135") (footprint "Package_SO:SOIC-16W_7.5x10.3mm_P1.27mm")
@@
       (reference "D14") (unit 1) (value "SN74AC08DR") (footprint "Package_SO:SOIC-14_3.9x8.7mm_P1.27mm")
     )
+    (path "/f75c0da5-ea98-45b1-9a07-415549f295ff/98cf1311-06d1-4b28-9e00-6c3437b1d954"
+      (reference "D15") (unit 1) (value "WRA1215S-3WR2") (footprint "Mornsun:WRA1215S-3WR2")
+    )
+    (path "/f75c0da5-ea98-45b1-9a07-415549f295ff/4fbb5034-268f-4ad1-9d51-05eeb29bb66f"
+      (reference "D16") (unit 1) (value "WRA1215S-3WR2") (footprint "Mornsun:WRA1215S-3WR2")
+    )
     (path "/83021f70-e61e-4ad3-bae7-b9f02b28be4f"
       (reference "H1") (unit 1) (value "MountingHole") (footprint "MountingHole:MountingHole_3.2mm_M3")
@@
       (reference "J33") (unit 1) (value "CH3") (footprint "SKiM459GD12E4 V2_smd:SKiM459GD12E4 V2_SMD_Pin")
     )
+    (path "/90ad37b3-1964-4d46-be98-f2e705808058/65c536fb-0128-4590-b82b-fdb4e26d7a6d"
+      (reference "Q1") (unit 1) (value "MJD44H11T4G") (footprint "Package_TO_SOT_SMD:TO-252-2")
+    )
+    (path "/90ad37b3-1964-4d46-be98-f2e705808058/8dccfa7b-9bb0-4338-ae96-3f72fc8cdc14"
+      (reference "Q2") (unit 1) (value "MJD45H11T4G") (footprint "Package_TO_SOT_SMD:TO-252-2")
+    )
+    (path "/90ad37b3-1964-4d46-be98-f2e705808058/dc1a99c1-443f-404d-ac5c-4039b2041de8"
+      (reference "Q3") (unit 1) (value "MJD44H11T4G") (footprint "Package_TO_SOT_SMD:TO-252-2")
+    )
+    (path "/90ad37b3-1964-4d46-be98-f2e705808058/93d9adb9-60b3-465f-8cea-435ddcdc3737"
+      (reference "Q4") (unit 1) (value "MJD45H11T4G") (footprint "Package_TO_SOT_SMD:TO-252-2")
+    )
     (path "/90ad37b3-1964-4d46-be98-f2e705808058/01e64fa8-c377-4fbf-9462-6f1ee162caf5"
       (reference "R1") (unit 1) (value "120") (footprint "Resistor_SMD:R_0805_2012Metric_Pad1.20x1.40mm_HandSolder")
@@
       (reference "R28") (unit 1) (value "120") (footprint "Resistor_SMD:R_0805_2012Metric_Pad1.20x1.40mm_HandSolder")
     )
+    (path "/90ad37b3-1964-4d46-be98-f2e705808058/8d4f131d-fa9f-4950-9005-b0558b9ba442"
+      (reference "R29") (unit 1) (value "3.9") (footprint "Resistor_SMD:R_2512_6332Metric_Pad1.40x3.35mm_HandSolder")
+    )
+    (path "/90ad37b3-1964-4d46-be98-f2e705808058/e93808f5-2a7e-497d-93a9-b6c73d933784"
+      (reference "R30") (unit 1) (value "3.9") (footprint "Resistor_SMD:R_2512_6332Metric_Pad1.40x3.35mm_HandSolder")
+    )
+    (path "/90ad37b3-1964-4d46-be98-f2e705808058/fd0bfc2c-c242-4c45-a2ce-a3cfcb0ffc5b"
+      (reference "R31") (unit 1) (value "10k") (footprint "Resistor_SMD:R_2512_6332Metric_Pad1.40x3.35mm_HandSolder")
+    )
+    (path "/90ad37b3-1964-4d46-be98-f2e705808058/00373f9d-a73f-483b-8b4a-b071819f2c6b"
+      (reference "R32") (unit 1) (value "10k") (footprint "Resistor_SMD:R_2512_6332Metric_Pad1.40x3.35mm_HandSolder")
+    )
   )

Commit message: Первая сырая расстановка, неполная
Parts:
- added J1: 2-338069-0, Connector_My:2-338069-0, symbol Connector_My:2-338069-0
Connections:
- new net +15V: J1.1, J1.2
- new net DCLINK_N: J1.4
- new net DCLINK_P: J1.3
- new net ERR: J1.15
- new net GND: J1.14, J1.16, J1.17, J1.18, J1.19, J1.20, J1.5, J1.6, J1.7
- new net HB1_BOT: J1.9
- new net HB1_TOP: J1.8
- new net HB2_BOT: J1.11
- new net HB2_TOP: J1.10
- new net HB3_BOT: J1.13
- new net HB3_TOP: J1.12
Other:
- sheet ADUM4135 renamed ADUM4135_1
- sheet Indication_ADUM renamed Indication_ADUM_1
- sheet Supply_Power renamed Supply_Power_1
- added sheet ADUM4135_2 (ADUM4135_2.kicad_sch)
- added sheet ADUM4135_3 (ADUM4135_3.kicad_sch)
- added sheet Common_ERR (Common_ERR.kicad_sch)
- added sheet DC_Measure (DC_Measure.kicad_sch)
- added sheet Indication_ADUM_2 (Indication_ADUM_2.kicad_sch)
- added sheet Indication_ADUM_3 (Indication_ADUM_3.kicad_sch)
- added sheet Logic_Protection_2 (Logic_Protection_2.kicad_sch)
- added sheet Logic_Protection_3 (Logic_Protection_3.kicad_sch)
- added sheet NTC_Handler (NTC_Handler.kicad_sch)
- added sheet Supply_Power_2 (Supply_Power_2.kicad_sch)
- added sheet Supply_Power_3 (Supply_Power_3.kicad_sch)
- added sheet Supply_Power_5V (Supply_Power_5V.kicad_sch)
- sheet Indication_ADUM_1: file Indication_ADUM.kicad_sch -> Indication_ADUM_1.kicad_sch
- sheet Supply_Power_1: file Supply_Power.kicad_sch -> Supply_Power_1.kicad_sch

Commit message: Почти финальная версия
Other:
- sheet NTC_Handler renamed PTC_Handler
- sheet PTC_Handler: file NTC_Handler.kicad_sch -> PTC_Handler.kicad_sch
Changed lines of the file:
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@@
     )
     (property "Value" "2-338069-0" (id 1) (at 235.204 121.92 0)
-      (effects (font (size 1.524 1.524)) (justify left))
+      (effects (font (size 1.524 1.524)) (justify left) hide)
     )
     (property "Footprint" "Connector_My:2-338069-0" (id 2) (at 231.394 151.892 0)
@@
     (stroke (width 0.1524) (type solid) (color 0 0 0 0))
     (fill (color 0 0 0 0.0000))
-    (property "Sheet name" "NTC_Handler" (id 0) (at 128.778 134.6704 0)
+    (property "Sheet name" "PTC_Handler" (id 0) (at 128.778 134.6704 0)
       (effects (font (size 1.27 1.27)) (justify left bottom))
     )
-    (property "Sheet file" "NTC_Handler.kicad_sch" (id 1) (at 128.778 158.3186 0)
+    (property "Sheet file" "PTC_Handler.kicad_sch" (id 1) (at 128.778 158.3186 0)
       (effects (font (size 1.27 1.27)) (justify left top))
     )
@@
       (reference "#PWR075") (unit 1) (value "GND") (footprint "")
     )
+    (path "/725fa47d-37a7-4087-9a93-0b03cc2ba810/bb3cfc38-db12-4f18-b194-10c63bf858b0"
+      (reference "#PWR076") (unit 1) (value "+5VD") (footprint "")
+    )
+    (path "/725fa47d-37a7-4087-9a93-0b03cc2ba810/5fb8c08d-5adb-4337-a579-4dc2d588a018"
+      (reference "#PWR077") (unit 1) (value "GND") (footprint "")
+    )
     (path "/a52110d1-8b82-46b9-820b-5e8319044e58/a2c44189-3d5f-461b-aba2-6162f21dea1f"
       (reference "#PWR079") (unit 1) (value "+15V") (footprint "")
@@
       (reference "C95") (unit 1) (value "100n") (footprint "Capacitor_SMD:C_0805_2012Metric_Pad1.18x1.45mm_HandSolder")
     )
+    (path "/725fa47d-37a7-4087-9a93-0b03cc2ba810/337ab399-74f7-497b-b869-aac45e5702d7"
+      (reference "C96") (unit 1) (value "0.1u") (footprint "Capacitor_SMD:C_0805_2012Metric_Pad1.18x1.45mm_HandSolder")
+    )
+    (path "/725fa47d-37a7-4087-9a93-0b03cc2ba810/597848f5-7df2-4cf2-ab54-aea6c747b2f5"
+      (reference "C97") (unit 1) (value "0.1u") (footprint "Capacitor_SMD:C_0805_2012Metric_Pad1.18x1.45mm_HandSolder")
+    )
+    (path "/725fa47d-37a7-4087-9a93-0b03cc2ba810/7b01af06-4f25-4987-95e9-617267432ecd"
+      (reference "C98") (unit 1) (value "0.1u") (footprint "Capacitor_SMD:C_0805_2012Metric_Pad1.18x1.45mm_HandSolder")
+    )
+    (path "/725fa47d-37a7-4087-9a93-0b03cc2ba810/8ac08bc0-d270-48d5-9d0a-b7435dbd84b8"
+      (reference "C99") (unit 1) (value "0.1u") (footprint "Capacitor_SMD:C_0805_2012Metric_Pad1.18x1.45mm_HandSolder")
+    )
+    (path "/725fa47d-37a7-4087-9a93-0b03cc2ba810/ff4c9bb3-25a4-4a69-aaac-c580cf2e9065"
+      (reference "C100") (unit 1) (value "0.1u") (footprint "Capacitor_SMD:C_0805_2012Metric_Pad1.18x1.45mm_HandSolder")
+    )
     (path "/90ad37b3-1964-4d46-be98-f2e705808058/89aad84a-99b2-4cff-9a18-0bcef9ff760f"
       (reference "D1") (unit 1) (value "ADUM4135") (footprint "Package_SO:SOIC-16W_7.5x10.3mm_P1.27mm")
@@
       (reference "R137") (unit 1) (value "10k") (footprint "Resistor_SMD:R_0805_2012Metric_Pad1.20x1.40mm_HandSolder")
     )
+    (path "/725fa47d-37a7-4087-9a93-0b03cc2ba810/442ca7f4-6834-475f-987c-b2917e7678db"
+      (reference "R138") (unit 1) (value "120") (footprint "Resistor_SMD:R_0805_2012Metric_Pad1.20x1.40mm_HandSolder")
+    )
+    (path "/725fa47d-37a7-4087-9a93-0b03cc2ba810/94077241-0a98-44d5-9df6-db4e2a083d31"
+      (reference "R139") (unit 1) (value "120") (footprint "Resistor_SMD:R_0805_2012Metric_Pad1.20x1.40mm_HandSolder")
+    )
+    (path "/725fa47d-37a7-4087-9a93-0b03cc2ba810/4d1d0761-a5e1-4fb0-adbf-44f9db81663e"
+      (reference "R140") (unit 1) (value "1.8k") (footprint "Resistor_SMD:R_0805_2012Metric_Pad1.20x1.40mm_HandSolder")
+    )
     (path "/b341ba61-0db2-4720-ae65-a3ee3f0accba/19518dde-0f07-4d38-937f-1ddd72089aa1"
       (reference "U1") (unit 1) (value "LM2904") (footprint "Package_SO:SO-8_3.9x4.9mm_P1.27mm")
@@
       (reference "U2") (unit 1) (value "R-785.0-1.0") (footprint "Converter_DCDC:Converter_DCDC_RECOM_R-78E-0.5_THT")
     )
-  )
+    (path "/725fa47d-37a7-4087-9a93-0b03cc2ba810/65a075e7-2b98-49ef-b105-7c6945abe096"
+      (reference "U3") (unit 1) (value "LM397") (footprint "Package_TO_SOT_SMD:SOT-23-5")
+    )
+    (path "/725fa47d-37a7-4087-9a93-0b03cc2ba810/3f2bd1b2-9b9a-4f4e-b16b-a5cb1869a7c9"
+      (reference "U4") (unit 1) (value "HCPL-0611") (footprint "Package_SO:SOIC-8_3.9x4.9mm_P1.27mm")
+    )
+  )

Commit message: Исправил ошибки, добавил резисторы в затвор, ревизия 2.0
Parts:
- H1, H10, H2, H3, H4, H5, H6, H7, H8, H9: footprint MountingHole:MountingHole_3.2mm_M3 -> Mounting_Hole_My:M3
- H11, H12: footprint MountingHole:MountingHole_4.3mm_M4 -> Mounting_Hole_My:M4
Connections:
- net NTC1_A renamed PTC1_A
- net NTC1_B renamed PTC1_B
- net NTC2_A renamed PTC2_A
- net NTC2_B renamed PTC2_B
- net NTC3_A renamed PTC3_A
- net NTC3_B renamed PTC3_B
