File: PTC_Handler.kicad_sch (KiCad schematic)
At the start: 10 parts, among them U3 LM397, U4 HCPL-0611

Commit message: Добавил названия элементов в схеме
Parts:
- added R142: 350, Resistor_SMD:R_0805_2012Metric_Pad1.20x1.40mm_HandSolder, symbol Device:R_Small
- gave numbers to parts that had none: 1
Connections:
- net +5VD: now also R142.1
- net RST_H1: now also R142.2
Other:
- moved on the sheet: C100
Changed lines of the file:
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@@
   (junction (at 116.84 109.22) (diameter 0) (color 0 0 0 0)
   )
+  (junction (at 204.47 91.44) (diameter 0) (color 0 0 0 0)
+  )
   (junction (at 197.485 108.585) (diameter 0) (color 0 0 0 0)
   )
@@
   (junction (at 144.78 93.98) (diameter 0) (color 0 0 0 0)
   )
+  (junction (at 197.485 96.52) (diameter 0) (color 0 0 0 0)
+  )
   (wire (pts (xy 144.78 93.98) (xy 144.78 101.6))
     (stroke (width 0) (type default) (color 0 0 0 0))
@@
     (stroke (width 0) (type default) (color 0 0 0 0))
   )
-  (wire (pts (xy 208.28 93.98) (xy 208.28 91.44))
-    (stroke (width 0) (type default) (color 0 0 0 0))
-  )
-  (wire (pts (xy 208.28 99.06) (xy 208.28 101.6))
+  (wire (pts (xy 197.485 96.52) (xy 198.755 96.52))
+    (stroke (width 0) (type default) (color 0 0 0 0))
+  )
+  (wire (pts (xy 212.09 101.6) (xy 212.09 99.06))
     (stroke (width 0) (type default) (color 0 0 0 0))
   )
@@
     (stroke (width 0) (type default) (color 0 0 0 0))
   )
+  (wire (pts (xy 212.09 91.44) (xy 212.09 93.98))
+    (stroke (width 0) (type default) (color 0 0 0 0))
+  )
   (wire (pts (xy 116.84 109.22) (xy 124.46 109.22))
     (stroke (width 0) (type default) (color 0 0 0 0))
@@
     (stroke (width 0) (type default) (color 0 0 0 0))
   )
-  (wire (pts (xy 193.04 91.44) (xy 208.28 91.44))
+  (wire (pts (xy 193.04 91.44) (xy 204.47 91.44))
     (stroke (width 0) (type default) (color 0 0 0 0))
   )
@@
     (stroke (width 0) (type default) (color 0 0 0 0))
   )
+  (wire (pts (xy 203.835 96.52) (xy 204.47 96.52))
+    (stroke (width 0) (type default) (color 0 0 0 0))
+  )
   (wire (pts (xy 124.46 93.98) (xy 144.78 93.98))
     (stroke (width 0) (type default) (color 0 0 0 0))
   )
+  (wire (pts (xy 204.47 91.44) (xy 212.09 91.44))
+    (stroke (width 0) (type default) (color 0 0 0 0))
+  )
   (wire (pts (xy 124.46 91.44) (xy 124.46 93.98))
     (stroke (width 0) (type default) (color 0 0 0 0))
@@
     (stroke (width 0) (type default) (color 0 0 0 0))
   )
-  (wire (pts (xy 193.04 101.6) (xy 208.28 101.6))
+  (wire (pts (xy 193.04 101.6) (xy 212.09 101.6))
     (stroke (width 0) (type default) (color 0 0 0 0))
   )
@@
   )
   (wire (pts (xy 200.025 108.585) (xy 197.485 108.585))
+    (stroke (width 0) (type default) (color 0 0 0 0))
+  )
+  (wire (pts (xy 204.47 96.52) (xy 204.47 91.44))
     (stroke (width 0) (type default) (color 0 0 0 0))
   )
@@
     )
     (property "Datasheet" "~" (id 3) (at 116.84 96.52 0)
+      (effects (font (size 1.27 1.27)) hide)
+    )
+    (pin "1")
+    (pin "2")
+  )
+  (symbol (lib_id "Device:R_Small") (at 201.295 96.52 270) (unit 1)
+    (in_bom yes) (on_board yes)
+    (property "Reference" "R142" (id 0) (at 201.295 94.615 90))
+    (property "Value" "350" (id 1) (at 201.295 98.171 90))
+    (property "Footprint" "Resistor_SMD:R_0805_2012Metric_Pad1.20x1.40mm_HandSolder" (id 2) (at 201.295 96.52 0)
+      (effects (font (size 1.27 1.27)) hide)
+    )
+    (property "Datasheet" "~" (id 3) (at 201.295 96.52 0)
       (effects (font (size 1.27 1.27)) hide)
     )
@@
   (symbol (lib_id "Device:R_Small") (at 164.465 83.82 270) (unit 1)
     (in_bom yes) (on_board yes)
-    (property "Reference" "R?" (id 0) (at 164.465 81.915 90))
+    (property "Reference" "R141" (id 0) (at 164.465 81.915 90))
     (property "Value" "300" (id 1) (at 164.465 85.471 90))
     (property "Footprint" "Resistor_SMD:R_0805_2012Metric_Pad1.20x1.40mm_HandSolder" (id 2) (at 164.465 83.82 0)
@@
     (pin "2")
   )
-  (symbol (lib_id "Device:C_Small") (at 208.28 96.52 0) (unit 1)
-    (in_bom yes) (on_board yes)
-    (property "Reference" "C100" (id 0) (at 202.565 94.615 0)
+  (symbol (lib_id "Device:C_Small") (at 212.09 96.52 0) (unit 1)
+    (in_bom yes) (on_board yes)
+    (property "Reference" "C100" (id 0) (at 206.375 94.615 0)
       (effects (font (size 1.27 1.27)) (justify left))
     )
-    (property "Value" "0.1u" (id 1) (at 207.645 98.425 0)
+    (property "Value" "0.1u" (id 1) (at 211.455 98.425 0)
       (effects (font (size 1.27 1.27)) (justify right))
     )
-    (property "Footprint" "Capacitor_SMD:C_0805_2012Metric_Pad1.18x1.45mm_HandSolder" (id 2) (at 208.28 96.52 0)
-      (effects (font (size 1.27 1.27)) hide)
-    )
-    (property "Datasheet" "~" (id 3) (at 208.28 96.52 0)
-      (effects (font (size 1.27 1.27)) hide)
-    )
+    (property "Footprint" "Capacitor_SMD:C_0805_2012Metric_Pad1.18x1.45mm_HandSolder" (id 2) (at 212.09 96.52 0)
+      (effects (font (size 1.27 1.27)) hide)
+    )
+    (property "Datasheet" "~" (id 3) (at 212.09 96.52 0)
+      (effects (font (size 1.27 1.27)) hide)
+    )

Commit message: Исправил ошибки, добавил резисторы в затвор, ревизия 2.0
Parts:
- R139: value 1k -> 1.8k
- R140: value 1.8k -> 1k
- R141: value 300 -> 1.5k
Connections:
- net +15V_L2: no longer R138.2
- net EL2: now also R138.1
- net NTC2_A renamed PTC2_B
- net PTC2_B: now also R138.2; no longer R138.1
Other:
- moved on the sheet: R138
Changed lines of the file:
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@@
   (junction (at 197.485 114.935) (diameter 0) (color 0 0 0 0)
   )
+  (junction (at 124.206 83.82) (diameter 0) (color 0 0 0 0)
+  )
   (junction (at 137.16 99.06) (diameter 0) (color 0 0 0 0)
   )
   (junction (at 132.08 109.22) (diameter 0) (color 0 0 0 0)
   )
+  (junction (at 124.206 93.98) (diameter 0) (color 0 0 0 0)
+  )
   (junction (at 116.84 83.82) (diameter 0) (color 0 0 0 0)
   )
@@
   (junction (at 152.4 83.82) (diameter 0) (color 0 0 0 0)
   )
-  (junction (at 124.46 109.22) (diameter 0) (color 0 0 0 0)
-  )
   (junction (at 197.485 105.41) (diameter 0) (color 0 0 0 0)
   )
   (junction (at 197.485 118.11) (diameter 0) (color 0 0 0 0)
   )
-  (junction (at 124.46 83.82) (diameter 0) (color 0 0 0 0)
-  )
   (junction (at 193.04 91.44) (diameter 0) (color 0 0 0 0)
   )
-  (junction (at 124.46 93.98) (diameter 0) (color 0 0 0 0)
-  )
   (junction (at 137.16 109.22) (diameter 0) (color 0 0 0 0)
   )
@@
   (junction (at 132.08 83.82) (diameter 0) (color 0 0 0 0)
   )
+  (junction (at 124.206 109.22) (diameter 0) (color 0 0 0 0)
+  )
   (junction (at 197.485 111.76) (diameter 0) (color 0 0 0 0)
   )
@@
     (stroke (width 0) (type default) (color 0 0 0 0))
   )
+  (wire (pts (xy 109.474 88.9) (xy 124.206 88.9))
+    (stroke (width 0) (type default) (color 0 0 0 0))
+  )
   (wire (pts (xy 197.485 118.11) (xy 197.485 121.285))
     (stroke (width 0) (type default) (color 0 0 0 0))
@@
     (stroke (width 0) (type default) (color 0 0 0 0))
   )
-  (wire (pts (xy 116.84 109.22) (xy 124.46 109.22))
-    (stroke (width 0) (type default) (color 0 0 0 0))
-  )
   (wire (pts (xy 144.78 93.98) (xy 147.32 93.98))
     (stroke (width 0) (type default) (color 0 0 0 0))
@@
     (stroke (width 0) (type default) (color 0 0 0 0))
   )
-  (wire (pts (xy 124.46 83.82) (xy 124.46 86.36))
+  (wire (pts (xy 124.206 83.82) (xy 132.08 83.82))
     (stroke (width 0) (type default) (color 0 0 0 0))
   )
@@
     (stroke (width 0) (type default) (color 0 0 0 0))
   )
-  (wire (pts (xy 124.46 93.98) (xy 144.78 93.98))
-    (stroke (width 0) (type default) (color 0 0 0 0))
-  )
   (wire (pts (xy 204.47 91.44) (xy 212.09 91.44))
     (stroke (width 0) (type default) (color 0 0 0 0))
   )
-  (wire (pts (xy 124.46 91.44) (xy 124.46 93.98))
+  (wire (pts (xy 124.206 109.22) (xy 132.08 109.22))
     (stroke (width 0) (type default) (color 0 0 0 0))
   )
@@
     (stroke (width 0) (type default) (color 0 0 0 0))
   )
-  (wire (pts (xy 124.46 93.98) (xy 124.46 101.6))
+  (wire (pts (xy 124.206 101.854) (xy 124.206 93.98))
+    (stroke (width 0) (type default) (color 0 0 0 0))
+  )
+  (wire (pts (xy 109.474 91.694) (xy 124.206 91.694))
     (stroke (width 0) (type default) (color 0 0 0 0))
   )
@@
     (stroke (width 0) (type default) (color 0 0 0 0))
   )
+  (wire (pts (xy 124.206 91.694) (xy 124.206 93.98))
+    (stroke (width 0) (type default) (color 0 0 0 0))
+  )
+  (wire (pts (xy 124.206 93.98) (xy 144.78 93.98))
+    (stroke (width 0) (type default) (color 0 0 0 0))
+  )
   (wire (pts (xy 197.485 111.76) (xy 197.485 108.585))
     (stroke (width 0) (type default) (color 0 0 0 0))
@@
     (stroke (width 0) (type default) (color 0 0 0 0))
   )
-  (wire (pts (xy 109.22 104.14) (xy 124.46 104.14))
-    (stroke (width 0) (type default) (color 0 0 0 0))
-  )
   (wire (pts (xy 190.5 93.98) (xy 193.04 93.98))
     (stroke (width 0) (type default) (color 0 0 0 0))
@@
     (stroke (width 0) (type default) (color 0 0 0 0))
   )
+  (wire (pts (xy 124.206 106.934) (xy 124.206 109.22))
+    (stroke (width 0) (type default) (color 0 0 0 0))
+  )
   (wire (pts (xy 193.04 91.44) (xy 193.04 88.9))
     (stroke (width 0) (type default) (color 0 0 0 0))
@@
     (stroke (width 0) (type default) (color 0 0 0 0))
   )
-  (wire (pts (xy 124.46 104.14) (xy 124.46 109.22))
+  (wire (pts (xy 124.206 83.82) (xy 124.206 88.9))
     (stroke (width 0) (type default) (color 0 0 0 0))
   )
@@
     (stroke (width 0) (type default) (color 0 0 0 0))
   )
-  (wire (pts (xy 109.22 101.6) (xy 124.46 101.6))
-    (stroke (width 0) (type default) (color 0 0 0 0))
-  )
   (wire (pts (xy 190.5 96.52) (xy 197.485 96.52))
     (stroke (width 0) (type default) (color 0 0 0 0))
@@
     (stroke (width 0) (type default) (color 0 0 0 0))
   )
-  (wire (pts (xy 124.46 83.82) (xy 132.08 83.82))
-    (stroke (width 0) (type default) (color 0 0 0 0))
-  )
-  (wire (pts (xy 124.46 109.22) (xy 132.08 109.22))
+  (wire (pts (xy 116.84 83.82) (xy 124.206 83.82))
+    (stroke (width 0) (type default) (color 0 0 0 0))
+  )
+  (wire (pts (xy 116.84 109.22) (xy 124.206 109.22))
     (stroke (width 0) (type default) (color 0 0 0 0))
   )
@@
     (stroke (width 0) (type default) (color 0 0 0 0))
   )
-  (wire (pts (xy 116.84 83.82) (xy 124.46 83.82))
-    (stroke (width 0) (type default) (color 0 0 0 0))
-  )
   (wire (pts (xy 116.84 83.82) (xy 116.84 93.98))
     (stroke (width 0) (type default) (color 0 0 0 0))
@@
     )
   )
-  (global_label "NTC2_A" (shape input) (at 109.22 101.6 180) (fields_autoplaced)
+  (global_label "PTC2_A" (shape input) (at 109.474 88.9 180) (fields_autoplaced)
     (effects (font (size 1.27 1.27)) (justify right))
-    (property "Intersheet References" "${INTERSHEET_REFS}" (id 0) (at 99.9731 101.5206 0)
+    (property "Intersheet References" "${INTERSHEET_REFS}" (id 0) (at 100.2876 88.8206 0)
       (effects (font (size 1.27 1.27)) (justify right) hide)
     )
@@
     )
   )
-  (global_label "NTC2_B" (shape input) (at 109.22 104.14 180) (fields_autoplaced)
+  (global_label "PTC2_B" (shape input) (at 109.474 91.694 180) (fields_autoplaced)
     (effects (font (size 1.27 1.27)) (justify right))
-    (property "Intersheet References" "${INTERSHEET_REFS}" (id 0) (at 99.7917 104.0606 0)
+    (property "Intersheet References" "${INTERSHEET_REFS}" (id 0) (at 100.1061 91.6146 0)
       (effects (font (size 1.27 1.27)) (justify right) hide)
     )
@@
     (pin "8")
   )
-  (symbol (lib_id "Device:R_Small") (at 124.46 88.9 180) (unit 1)
-    (in_bom yes) (on_board yes)
-    (property "Reference" "R138" (id 0) (at 121.285 86.36 0))
-    (property "Value" "1k" (id 1) (at 121.92 88.9 0))
-    (property "Footprint" "Resistor_SMD:R_0805_2012Metric_Pad1.20x1.40mm_HandSolder" (id 2) (at 124.46 88.9 0)
-      (effects (font (size 1.27 1.27)) hide)
-    )
-    (property "Datasheet" "~" (id 3) (at 124.46 88.9 0)
+  (symbol (lib_id "Device:R_Small") (at 124.206 104.394 180) (unit 1)
+    (in_bom yes) (on_board yes)
+    (property "Reference" "R138" (id 0) (at 120.396 102.87 0))
+    (property "Value" "1k" (id 1) (at 121.666 105.41 0))
+    (property "Footprint" "Resistor_SMD:R_0805_2012Metric_Pad1.20x1.40mm_HandSolder" (id 2) (at 124.206 104.394 0)
+      (effects (font (size 1.27 1.27)) hide)
+    )
+    (property "Datasheet" "~" (id 3) (at 124.206 104.394 0)
       (effects (font (size 1.27 1.27)) hide)
     )
@@
     (in_bom yes) (on_board yes)
     (property "Reference" "R140" (id 0) (at 128.27 102.87 0))
-    (property "Value" "1.8k" (id 1) (at 128.905 105.41 0))
+    (property "Value" "1k" (id 1) (at 128.905 105.41 0))
     (property "Footprint" "Resistor_SMD:R_0805_2012Metric_Pad1.20x1.40mm_HandSolder" (id 2) (at 132.08 104.14 0)
       (effects (font (size 1.27 1.27)) hide)
@@
   (symbol (lib_id "Device:R_Small") (at 132.08 88.9 180) (unit 1)
     (in_bom yes) (on_board yes)
-    (property "Reference" "R139" (id 0) (at 128.905 86.36 0))
-    (property "Value" "1k" (id 1) (at 129.54 88.9 0))
+    (property "Reference" "R139" (id 0) (at 128.27 87.63 0))
+    (property "Value" "1.8k" (id 1) (at 128.778 90.17 0))
     (property "Footprint" "Resistor_SMD:R_0805_2012Metric_Pad1.20x1.40mm_HandSolder" (id 2) (at 132.08 88.9 0)
       (effects (font (size 1.27 1.27)) hide)
@@
     (in_bom yes) (on_board yes)
     (property "Reference" "R141" (id 0) (at 164.465 81.915 90))
-    (property "Value" "300" (id 1) (at 164.465 85.471 90))
+    (property "Value" "1.5k" (id 1) (at 164.465 85.471 90))
     (property "Footprint" "Resistor_SMD:R_0805_2012Metric_Pad1.20x1.40mm_HandSolder" (id 2) (at 164.465 83.82 0)
       (effects (font (size 1.27 1.27)) hide)

Commit message: Версия для резонита REV2.1
Parts:
- R141: value 1.5k -> 350
Changed lines of the file:
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@@
     (in_bom yes) (on_board yes)
     (property "Reference" "R141" (id 0) (at 164.465 81.915 90))
-    (property "Value" "1.5k" (id 1) (at 164.465 85.471 90))
+    (property "Value" "350" (id 1) (at 164.465 85.471 90))
     (property "Footprint" "Resistor_SMD:R_0805_2012Metric_Pad1.20x1.40mm_HandSolder" (id 2) (at 164.465 83.82 0)
       (effects (font (size 1.27 1.27)) hide)
