File: ADUM4135.kicad_sch (KiCad schematic)
At the start: 24 parts

Commit message: Одна стойка
Parts:
- added C21, C22, C27, C28: 1u, Capacitor_SMD:C_0805_2012Metric_Pad1.18x1.45mm_HandSolder, symbol Device:C_Small
- added Q1, Q3: MJD44H11T4G, Package_TO_SOT_SMD:TO-252-2, symbol Transistor_BJT:BCP56
- added Q2, Q4: MJD45H11T4G, Package_TO_SOT_SMD:TO-252-2, symbol Transistor_BJT:2SB817
- added R29, R30: 3.9, Resistor_SMD:R_2512_6332Metric_Pad1.40x3.35mm_HandSolder, symbol Device:R_Small
- added R31, R32: 10k, Resistor_SMD:R_2512_6332Metric_Pad1.40x3.35mm_HandSolder, symbol Device:R_Small
Connections:
- net +15V_H1: now also C21.1, Q1.2 (C), Q1.4 (C)
- net +15V_L1: now also C27.1, Q3.2 (C), Q3.4 (C)
- net EL1: now also C27.2, C28.1
- net GH1: now also R29.1, R31.1; no longer D1.15 (GATE_SENSE), R2.1, R3.1
- net GL1: now also R30.1, R32.1; no longer D4.15 (GATE_SENSE), R8.1, R9.1
- net OUT1: now also C21.2, C22.1
- net -8V_H1 renamed -15V_H1
- net -15V_H1: now also C22.2, Q2.2 (C), R31.2
- net -8V_L1 renamed -15V_L1
- net -15V_L1: now also C28.2, Q4.2 (C), R32.2
- new net: Q1.3 (E), Q2.3 (E), R29.2
- new net: Q3.3 (E), Q4.3 (E), R30.2
- new net BH1_CLOSE: Q1.1 (B), Q2.1 (B), R2.1, R3.1
- new net BL1_CLOSE: Q3.1 (B), Q4.1 (B), R8.1, R9.1
- no-connect marks 0 -> 2
Other:
- moved on the sheet: C3, C4, C5, C6, D2, D3, D4, D5, D6, R10, R11, R12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

Commit message: Первая сырая расстановка, неполная
Parts:
- R31, R32: footprint Resistor_SMD:R_2512_6332Metric_Pad1.40x3.35mm_HandSolder -> Resistor_SMD:R_1210_3225Metric_Pad1.30x2.65mm_HandSolder
Connections:
- net -15V_H1: no longer R31.2
- net -15V_L1: no longer R32.2
- net EL1: now also R32.2
- net OUT1: now also R31.2
- net GND3 renamed GND
Other:
- moved on the sheet: R31, R32

Commit message: Добавил названия элементов в схеме
Parts:
- D2, D6: value US3M-13 -> MURS360T3G
- D3, D5: value BZT52C10-7-F -> MMSZ5240B
Changed lines of the file:
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@@
     (in_bom yes) (on_board yes)
     (property "Reference" "D2" (id 0) (at 122.682 82.804 90))
-    (property "Value" "US3M-13" (id 1) (at 117.856 83.566 0)
+    (property "Value" "MURS360T3G" (id 1) (at 117.856 83.566 0)
       (effects (font (size 1.27 1.27)) hide)
     )
@@
       (effects (font (size 1.27 1.27)) (justify left))
     )
-    (property "Value" "BZT52C10-7-F" (id 1) (at 113.538 161.798 0)
+    (property "Value" "MMSZ5240B" (id 1) (at 113.538 161.798 0)
       (effects (font (size 1.27 1.27)) (justify left))
     )
@@
       (effects (font (size 1.27 1.27)) (justify left))
     )
-    (property "Value" "BZT52C10-7-F" (id 1) (at 114.046 82.804 90)
+    (property "Value" "MMSZ5240B" (id 1) (at 114.046 82.804 90)
       (effects (font (size 1.27 1.27)) (justify left) hide)
     )
@@
     (in_bom yes) (on_board yes)
     (property "Reference" "D6" (id 0) (at 129.032 148.336 0))
-    (property "Value" "US3M-13" (id 1) (at 129.794 153.162 0))
+    (property "Value" "MURS360T3G" (id 1) (at 129.794 153.162 0))
     (property "Footprint" "Diode_SMD:D_SMC" (id 2) (at 129.032 150.622 90)
       (effects (font (size 1.27 1.27)) hide)

Commit message: Исправил ошибки, добавил резисторы в затвор, ревизия 2.0
Parts:
- added R143, R146: 3.9, Resistor_SMD:R_2512_6332Metric_Pad1.40x3.35mm_HandSolder, symbol Device:R_Small
- R2, R3, R8, R9: footprint Resistor_SMD:R_2512_6332Metric_Pad1.40x3.35mm_HandSolder -> Resistor_SMD:R_1210_3225Metric_Pad1.30x2.65mm_HandSolder
Connections:
- net GH1: now also R143.1
- net GL1: now also R146.1
- net at Q1.3 (E), Q2.3 (E), R29.2: now also R143.2
- net at Q3.3 (E), Q4.3 (E), R30.2: now also R146.2
Other:
- moved on the sheet: R29, R30

Commit message: Версия для резонита REV2.1
Parts:
- removed R11, R6: 2.2k, Resistor_SMD:R_0805_2012Metric_Pad1.20x1.40mm_HandSolder, symbol Device:R_Small
Changed lines of the file:
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@@
   (junction (at 60.198 61.722) (diameter 0) (color 0 0 0 0)
-  )
-  (junction (at 120.396 65.532) (diameter 0) (color 0 0 0 0)
   )
   (junction (at 59.944 146.812) (diameter 0) (color 0 0 0 0)
@@
     (stroke (width 0) (type default) (color 0 0 0 0))
   )
-  (wire (pts (xy 115.824 145.796) (xy 112.776 145.796))
-    (stroke (width 0) (type default) (color 0 0 0 0))
-  )
   (wire (pts (xy 154.686 58.674) (xy 155.956 58.674))
     (stroke (width 0) (type default) (color 0 0 0 0))
@@
     (stroke (width 0) (type default) (color 0 0 0 0))
   )
-  (wire (pts (xy 129.032 65.532) (xy 120.396 65.532))
-    (stroke (width 0) (type default) (color 0 0 0 0))
-  )
   (wire (pts (xy 126.746 126.238) (xy 126.746 127))
     (stroke (width 0) (type default) (color 0 0 0 0))
@@
     (stroke (width 0) (type default) (color 0 0 0 0))
   )
-  (wire (pts (xy 125.984 143.764) (xy 128.778 143.764))
-    (stroke (width 0) (type default) (color 0 0 0 0))
-  )
   (wire (pts (xy 129.032 159.258) (xy 132.588 159.258))
     (stroke (width 0) (type default) (color 0 0 0 0))
@@
     (stroke (width 0) (type default) (color 0 0 0 0))
   )
-  (wire (pts (xy 115.824 143.764) (xy 120.904 143.764))
-    (stroke (width 0) (type default) (color 0 0 0 0))
-  )
   (wire (pts (xy 162.814 52.324) (xy 155.956 52.324))
     (stroke (width 0) (type default) (color 0 0 0 0))
@@
     (stroke (width 0) (type default) (color 0 0 0 0))
   )
-  (wire (pts (xy 129.032 79.756) (xy 129.032 82.55))
-    (stroke (width 0) (type default) (color 0 0 0 0))
-  )
   (wire (pts (xy 97.536 139.192) (xy 102.616 139.192))
     (stroke (width 0) (type default) (color 0 0 0 0))
   )
-  (wire (pts (xy 129.032 74.676) (xy 129.032 65.532))
-    (stroke (width 0) (type default) (color 0 0 0 0))
-  )
   (wire (pts (xy 184.912 56.134) (xy 186.69 56.134))
     (stroke (width 0) (type default) (color 0 0 0 0))
@@
     (stroke (width 0) (type default) (color 0 0 0 0))
   )
-  (wire (pts (xy 115.824 145.796) (xy 115.824 143.764))
-    (stroke (width 0) (type default) (color 0 0 0 0))
-  )
   (wire (pts (xy 191.77 146.812) (xy 190.5 146.812))
     (stroke (width 0) (type default) (color 0 0 0 0))
@@
   )
   (wire (pts (xy 120.396 79.756) (xy 120.396 80.264))
-    (stroke (width 0) (type default) (color 0 0 0 0))
-  )
-  (wire (pts (xy 112.776 145.796) (xy 112.776 150.622))
     (stroke (width 0) (type default) (color 0 0 0 0))
   )
@@
     )
   )
-  (global_label "+15V_H1" (shape input) (at 129.032 82.55 270) (fields_autoplaced)
-    (effects (font (size 1.27 1.27)) (justify right))
-    (property "Intersheet References" "${INTERSHEET_REFS}" (id 0) (at 129.1114 93.5507 90)
-      (effects (font (size 1.27 1.27)) (justify right) hide)
-    )
-  )
   (global_label "OUT1" (shape input) (at 194.564 68.834 0) (fields_autoplaced)
     (effects (font (size 1.27 1.27)) (justify left))
@@
     (effects (font (size 1.27 1.27)) (justify left))
     (property "Intersheet References" "${INTERSHEET_REFS}" (id 0) (at 109.1052 61.8014 0)
-      (effects (font (size 1.27 1.27)) (justify left) hide)
-    )
-  )
-  (global_label "+15V_L1" (shape input) (at 128.778 143.764 0) (fields_autoplaced)
-    (effects (font (size 1.27 1.27)) (justify left))
-    (property "Intersheet References" "${INTERSHEET_REFS}" (id 0) (at 139.4763 143.6846 0)
       (effects (font (size 1.27 1.27)) (justify left) hide)
     )
@@
     (pin "3")
     (pin "4")
-  )
-  (symbol (lib_id "Device:R_Small") (at 123.444 143.764 90) (unit 1)
-    (in_bom yes) (on_board yes)
-    (property "Reference" "R11" (id 0) (at 123.444 141.732 90))
-    (property "Value" "2.2k" (id 1) (at 123.444 145.796 90))
-    (property "Footprint" "Resistor_SMD:R_0805_2012Metric_Pad1.20x1.40mm_HandSolder" (id 2) (at 123.444 143.764 0)
-      (effects (font (size 1.27 1.27)) hide)
-    )
-    (property "Datasheet" "~" (id 3) (at 123.444 143.764 0)
-      (effects (font (size 1.27 1.27)) hide)
-    )
-    (pin "1")
-    (pin "2")
   )
   (symbol (lib_id "Device:D_Schottky_Small") (at 117.856 159.258 0) (unit 1)
@@
       (effects (font (size 1.27 1.27)) hide)
     )
-    (pin "1")
-    (pin "2")
-  )
-  (symbol (lib_id "Device:R_Small") (at 129.032 77.216 0) (unit 1)
-    (in_bom yes) (on_board yes)
-    (property "Reference" "R6" (id 0) (at 131.064 77.216 0))
-    (property "Value" "2.2k" (id 1) (at 127 77.216 90))
-    (property "Footprint" "Resistor_SMD:R_0805_2012Metric_Pad1.20x1.40mm_HandSolder" (id 2) (at 129.032 77.216 0)
-      (effects (font (size 1.27 1.27)) hide)
-    )
-    (property "Datasheet" "~" (id 3) (at 129.032 77.216 0)
-      (effects (font (size 1.27 1.27)) hide)
-    )

Commit message: Финальная версия для производства
Parts:
- R12, R4: value 0 -> 10k
- R143, R146, R29, R30: value 3.9 -> 3
- R2, R3, R8, R9: value 3.9 -> 50
Changed lines of the file:
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@@
     (in_bom yes) (on_board yes)
     (property "Reference" "R2" (id 0) (at 100.33 52.197 90))
-    (property "Value" "3.9" (id 1) (at 100.33 48.26 90))
+    (property "Value" "50" (id 1) (at 100.33 48.26 90))
     (property "Footprint" "Resistor_SMD:R_1210_3225Metric_Pad1.30x2.65mm_HandSolder" (id 2) (at 100.33 50.292 0)
       (effects (font (size 1.27 1.27)) hide)
@@
     (in_bom yes) (on_board yes)
     (property "Reference" "R9" (id 0) (at 100.076 144.907 90))
-    (property "Value" "3.9" (id 1) (at 100.076 140.97 90))
+    (property "Value" "50" (id 1) (at 100.076 140.97 90))
     (property "Footprint" "Resistor_SMD:R_1210_3225Metric_Pad1.30x2.65mm_HandSolder" (id 2) (at 100.076 143.002 0)
       (effects (font (size 1.27 1.27)) hide)
@@
     (in_bom yes) (on_board yes)
     (property "Reference" "R146" (id 0) (at 187.706 144.653 90))
-    (property "Value" "3.9" (id 1) (at 187.706 142.748 90))
+    (property "Value" "3" (id 1) (at 187.706 142.748 90))
     (property "Footprint" "Resistor_SMD:R_2512_6332Metric_Pad1.40x3.35mm_HandSolder" (id 2) (at 187.706 142.748 0)
       (effects (font (size 1.27 1.27)) hide)
@@
     (in_bom yes) (on_board yes)
     (property "Reference" "R4" (id 0) (at 122.682 77.216 0))
-    (property "Value" "0" (id 1) (at 118.364 77.216 90))
+    (property "Value" "10k" (id 1) (at 118.364 77.216 90))
     (property "Footprint" "Resistor_SMD:R_1206_3216Metric_Pad1.30x1.75mm_HandSolder" (id 2) (at 120.396 77.216 0)
       (effects (font (size 1.27 1.27)) hide)
@@
     (in_bom yes) (on_board yes)
     (property "Reference" "R12" (id 0) (at 123.444 148.336 90))
-    (property "Value" "0" (id 1) (at 123.444 153.162 90))
+    (property "Value" "10k" (id 1) (at 123.444 153.162 90))
     (property "Footprint" "Resistor_SMD:R_1206_3216Metric_Pad1.30x1.75mm_HandSolder" (id 2) (at 123.444 150.622 0)
       (effects (font (size 1.27 1.27)) hide)
@@
     (in_bom yes) (on_board yes)
     (property "Reference" "R29" (id 0) (at 182.372 58.039 90))
-    (property "Value" "3.9" (id 1) (at 182.372 56.134 90))
+    (property "Value" "3" (id 1) (at 182.372 56.134 90))
     (property "Footprint" "Resistor_SMD:R_2512_6332Metric_Pad1.40x3.35mm_HandSolder" (id 2) (at 182.372 56.134 0)
       (effects (font (size 1.27 1.27)) hide)
@@
     (in_bom yes) (on_board yes)
     (property "Reference" "D6" (id 0) (at 129.032 148.336 0))
-    (property "Value" "MURS360T3G" (id 1) (at 129.794 153.162 0))
+    (property "Value" "MURS360T3G" (id 1) (at 132.334 153.162 0))
     (property "Footprint" "Diode_SMD:D_SMC" (id 2) (at 129.032 150.622 90)
       (effects (font (size 1.27 1.27)) hide)
@@
     (in_bom yes) (on_board yes)
     (property "Reference" "R8" (id 0) (at 100.076 137.287 90))
-    (property "Value" "3.9" (id 1) (at 100.076 133.35 90))
+    (property "Value" "50" (id 1) (at 100.076 133.35 90))
     (property "Footprint" "Resistor_SMD:R_1210_3225Metric_Pad1.30x2.65mm_HandSolder" (id 2) (at 100.076 135.382 0)
       (effects (font (size 1.27 1.27)) hide)
@@
     (in_bom yes) (on_board yes)
     (property "Reference" "R3" (id 0) (at 100.33 59.817 90))
-    (property "Value" "3.9" (id 1) (at 100.33 55.88 90))
+    (property "Value" "50" (id 1) (at 100.33 55.88 90))
     (property "Footprint" "Resistor_SMD:R_1210_3225Metric_Pad1.30x2.65mm_HandSolder" (id 2) (at 100.33 57.912 0)
       (effects (font (size 1.27 1.27)) hide)
@@
     (in_bom yes) (on_board yes)
     (property "Reference" "R30" (id 0) (at 187.96 148.717 90))
-    (property "Value" "3.9" (id 1) (at 187.96 146.812 90))
+    (property "Value" "3" (id 1) (at 187.96 146.812 90))
     (property "Footprint" "Resistor_SMD:R_2512_6332Metric_Pad1.40x3.35mm_HandSolder" (id 2) (at 187.96 146.812 0)
       (effects (font (size 1.27 1.27)) hide)
@@
     (in_bom yes) (on_board yes)
     (property "Reference" "R143" (id 0) (at 182.372 63.627 90))
-    (property "Value" "3.9" (id 1) (at 182.372 61.722 90))
+    (property "Value" "3" (id 1) (at 182.372 61.722 90))
     (property "Footprint" "Resistor_SMD:R_2512_6332Metric_Pad1.40x3.35mm_HandSolder" (id 2) (at 182.372 61.722 0)
       (effects (font (size 1.27 1.27)) hide)
